Commit message: Added IK server and client with student code template

File: kinematics_project/kuka_arm/urdf/kr210.urdf.xacro (robot description, xacro)
@@ -265,5 +265,5 @@
     <child link="right_gripper_finger_link" />
     <axis xyz="0 1 0" />
-    <limit effort="100" lower="0.0" upper="0.06" velocity="0.05" />
+    <limit effort="100" lower="-0.01" upper="0.06" velocity="0.05" />
     <dynamics damping="0.7" />
   </joint>
@@ -273,5 +273,5 @@
     <child link="left_gripper_finger_link" />
     <axis xyz="0 -1 0" />
-    <limit effort="100" lower="0.0" upper="0.06" velocity="0.05" />
+    <limit effort="100" lower="-0.01" upper="0.06" velocity="0.05" />
     <dynamics damping="0.7" />
   </joint>

File: kinematics_project/kuka_arm/urdf/target.urdf.xacro (robot description, xacro)
@@ -10,5 +10,5 @@
       <geometry>
         <cylinder radius="0.05" length="0.25"/>
-        <box size="0.10 0.10 0.25"/>
+        <!--box size="0.10 0.10 0.25"/-->
       </geometry>
     </visual>
